File: 00_Clock and Power Supply/select-circuit.kicad_sch (KiCad schematic)
At the start: 4 parts, among them SW3 SW_SPDT, U4 74LS01

Commit message: Last revision of the cpu, all boards have been ordered. Implementation to be tested and documented in following commits.
Parts:
- removed U4: 74LS01, Package_DIP:DIP-14_W7.62mm, symbol 74xx:74LS01
- added TP5: Select, TestPoint:TestPoint_Loop_D3.50mm_Drill0.9mm_Beaded, symbol Connector:TestPoint
- added U4: 74LS00, Package_DIP:DIP-14_W7.62mm, symbol 74xx:74LS00
Connections:
- net GND: now also U4.7 (GND)
- net Select: now also TP5.1, U4.2, U4.6
- net VCC: now also U4.10, U4.12, U4.13, U4.14 (VCC), U4.9
- net at R8.1, SW3.1 (A): now also U4.1
- net at R9.1, SW3.3 (C): now also U4.5
- new net: U4.3, U4.4
