File: 00_Clock and Power Supply/stable-clock.kicad_sch (KiCad schematic)
At the start: 6 parts, among them SW2 SPST, U3 LM555xN

Commit message: Last revision of the cpu, all boards have been ordered. Implementation to be tested and documented in following commits.
Parts:
- added TP4: Stable, TestPoint:TestPoint_Loop_D3.50mm_Drill0.9mm_Beaded, symbol Connector:TestPoint
- renumbered C6 to C10, C7 to C11
Connections:
- net Stable: now also TP4.1
Changed lines of the file:
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@@
+	)
+	(junction
+		(at 172.72 88.9)
+		(diameter 0)
+		(color 0 0 0 0)
 	)
 	(junction
@@
 	(wire
 		(pts
+			(xy 172.72 88.9) (xy 175.26 88.9)
+		)
+		(stroke
+			(width 0)
+			(type default)
+		)
+	)
+	(wire
+		(pts
 			(xy 135.89 93.98) (xy 144.78 93.98)
 		)
@@
 	(wire
 		(pts
+			(xy 172.72 85.09) (xy 172.72 88.9)
+		)
+		(stroke
+			(width 0)
+			(type default)
+		)
+	)
+	(wire
+		(pts
 			(xy 157.48 76.2) (xy 187.96 76.2)
 		)
@@
 	(wire
 		(pts
-			(xy 170.18 88.9) (xy 173.99 88.9)
+			(xy 170.18 88.9) (xy 172.72 88.9)
 		)
 		(stroke
@@
 	(hierarchical_label "Stable"
 		(shape output)
-		(at 173.99 88.9 0)
+		(at 175.26 88.9 0)
 		(effects
 			(font
@@
 		(dnp no)
 		(fields_autoplaced yes)
-		(property "Reference" "C6"
+		(property "Reference" "C10"
 			(at 191.77 100.7109 0)
 			(effects
@@
 			(project "Clock and Power Supply"
 				(path "/dd2fa5d1-1d39-4336-8d0e-915c0713d390/6dbac2c2-5bf9-4152-89f2-bbea8d72f94c"
-					(reference "C6")
+					(reference "C10")
 					(unit 1)
 				)
@@
 		(dnp no)
 		(fields_autoplaced yes)
-		(property "Reference" "C7"
+		(property "Reference" "C11"
 			(at 139.7 105.4099 0)
 			(effects
@@
 			(project "Clock and Power Supply"
 				(path "/dd2fa5d1-1d39-4336-8d0e-915c0713d390/6dbac2c2-5bf9-4152-89f2-bbea8d72f94c"
-					(reference "C7")
+					(reference "C11")
 					(unit 1)
 				)
@@
 					(unit 1)
 				)
+			)
+		)
+	)
+	(symbol
+		(lib_id "Connector:TestPoint")
+		(at 172.72 85.09 0)
+		(unit 1)
+		(exclude_from_sim no)
+		(in_bom yes)
+		(on_board yes)
+		(dnp no)
+		(fields_autoplaced yes)
+		(property "Reference" "TP4"
+			(at 175.26 80.5179 0)
+			(effects
+				(font
+					(size 1.27 1.27)
+				)
+				(justify left)
+			)
+		)
+		(property "Value" "Stable"
+			(at 175.26 83.0579 0)
+			(effects
+				(font
+					(size 1.27 1.27)
+				)
+				(justify left)
+			)
+		)
+		(property "Footprint" "TestPoint:TestPoint_Loop_D3.50mm_Drill0.9mm_Beaded"
+			(at 177.8 85.09 0)
+			(effects
+				(font
+					(size 1.27 1.27)
+				)
+				(hide yes)
+			)
+		)
+		(property "Datasheet" "~"
+			(at 177.8 85.09 0)
+			(effects
+				(font
+					(size 1.27 1.27)
+				)
+				(hide yes)
+			)
+		)
+		(property "Description" "test point"
+			(at 172.72 85.09 0)
+			(effects
+				(font
+					(size 1.27 1.27)
+				)
+				(hide yes)
+			)
+		)
+		(pin "1"
+		)
+		(instances
+			(project "Clock and Power Supply"
+				(path "/dd2fa5d1-1d39-4336-8d0e-915c0713d390/6dbac2c2-5bf9-4152-89f2-bbea8d72f94c"
+					(reference "TP4")
+					(unit 1)
+				)
