File: 02_Count Registers/Count Registers.kicad_sch (KiCad schematic)
At the start: 8 parts, among them J1 Data bus, J2 Alu-X bus, J3 Alu-Y bus, J4 Input 1, J5 Input 2, U1 74LS139, U2 74LS04, U3 74LS08

Commit message: Last revision of the cpu, all boards have been ordered. Implementation to be tested and documented in following commits.
Parts:
- removed U2: 74LS04, Package_DIP:DIP-14_W7.62mm, symbol 74xx:74LS04
- added C1, C2, C3: 100nF, Capacitor_THT:C_Disc_D4.7mm_W2.5mm_P5.00mm, symbol Device:C
- added unit 2 of U1
- added unit 5 of U1
- added unit 3 of U1
- added unit 4 of U1
- added unit 5 of U3
- added unit 3 of U3
- added unit 4 of U3
- renumbered U3 to U1, U1 to U2
Connections:
- net IC2 is gone; now on net IC1: J4.7 (Pin_7)
- net JC2 is gone; now on net JC1: J5.4 (Pin_4)
- net CLK: no longer U3.10, U3.13, U3.2, U3.5
- net Count register I/~{WE}: now also U1.3; no longer U2.7 (O3)
- net Count register J/~{WE}: now also U1.11; no longer U2.9 (O3)
- net GND: now also U3.4, U3.5, C1.2, C2.2, C3.2, U1.7 (GND), U3.10, U3.12, U3.13, U3.7 (GND), U3.9; no longer U1.7 (GND)
- net IC0: now also J4.6 (Pin_6), U2.2 (A0); no longer J4.5 (Pin_5), U2.3 (A1)
- net IC1: now also U2.3 (A1); no longer J4.6 (Pin_6), U2.2 (A0)
- net JC0: now also J5.3 (Pin_3), U2.14 (A0); no longer J5.2 (Pin_2), U2.13 (A1)
- net JC1: now also U2.13 (A1); no longer J5.3 (Pin_3), U2.14 (A0)
- net VCC: now also C1.1, C2.1, C3.1, U1.14 (VCC), U3.14 (VCC); no longer U1.14 (VCC)
- net at U2.5 (O1): now also U1.4
- net Count register I/U/~{D}: now reaches U2.6 (O2)
- net Count register I/U/~{D}: now also U1.5
- net Count register J/U/~{D}: now reaches U2.10 (O2)
- net Count register J/U/~{D}: now also U1.10
- net at U3.1: now also U2.9 (O3), U1.13
- net at U2.11 (O1): now also U1.9
- net Count register I/DOWN: no longer names the net of U3.6
- net Count register I/UP renamed Word Selector/~{CLR}
- removed net Count register J/DOWN: U3.11
- removed net Count register J/UP: U3.8
- new net: U1.2, U2.7 (O3), U3.2
- new net Count register I/~{CE}: U1.6
- new net Count register J/~{CE}: U1.8
- new net ~{IRI}: J4.5 (Pin_5), U1.1
- new net ~{JRI}: J5.2 (Pin_2), U1.12
- no-connect marks 2 -> 5
Other:
- added sheet Word Selector (word-selector.kicad_sch)
- sheet Count register I ports: added CLK, U/~{D}, ~{OE}; removed CLR, DOWN, UP
- sheet Count register J ports: added CLK, U/~{D}, ~{OE}; removed CLR, DOWN, UP
- note added: "Decoupling cap"
- note added: "ERC"
- note added: "Unsed Ports"
- moved on the sheet: J1, J2, J3, J4, J5, U2A, U2B, U2C
