File: 02_Count Registers/count_register.kicad_sch (KiCad schematic)
At the start: 19 parts, among them U5 74LS193, U6 74LS245, U7 74LS193

Commit message: Last revision of the cpu, all boards have been ordered. Implementation to be tested and documented in following commits.
Parts:
- removed U5, U7: 74LS193, Package_DIP:DIP-16_W7.62mm, symbol 74xx:74LS193
- added C4, C5, C6: 10nF, Capacitor_THT:C_Disc_D4.7mm_W2.5mm_P5.00mm, symbol Device:C
- added U4, U6: 74LS169, Package_DIP:DIP-16_W7.62mm, symbol 74xx:74LS169
- renumbered U6 to U5
Connections:
- net D0: now also U4.3 (P0)
- net D1: now also U4.4 (P1)
- net D2: now also U4.5 (P2)
- net D3: now also U4.6 (P3)
- net D4: now also U6.3 (P0)
- net D5: now also U6.4 (P1)
- net D6: now also U6.5 (P2)
- net D7: now also U6.6 (P3)
- net GND: now also C4.2, C5.2, C6.2, U4.10 (~{CET}), U4.8 (GND), U6.8 (GND)
- net Q0: now also U4.14 (Q0)
- net Q1: now also U4.13 (Q1)
- net Q2: now also U4.12 (Q2)
- net Q3: now also U4.11 (Q3)
- net Q4: now also U6.14 (Q0)
- net Q5: now also U6.13 (Q1)
- net Q6: now also U6.12 (Q2)
- net Q7: now also U6.11 (Q3)
- net VCC: now also C4.1, C5.1, C6.1, U4.16 (VCC), U6.16 (VCC)
- net ~{CE}: now also U4.7 (~{CEP}), U6.7 (~{CEP}); no longer U5.19 (~{CE})
- net ~{WE}: now also U4.9 (~{PE}), U6.9 (~{PE})
- new net: U4.15 (~{TC}), U6.10 (~{CET})
- new net CLK: U4.2 (CP), U6.2 (CP)
- new net U/~{D}: U4.1 (U/~{D}), U6.1 (U/~{D})
- new net ~{OE}: U5.19 (~{CE})
- no-connect marks 2 -> 1
Other:
- note added: "Decoupling cap"
- note added: "Out driver"
- title: Generic Register -> Count Register
- moved on the sheet: D1, D2, D3, D4, D5, D6, D7, D8, R1, R2, R3, R4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
