File: 03_Shift Registers/shift_register.kicad_sch (KiCad schematic)
At the start: 19 parts, among them U1 74LS194, U2 74LS245, U3 74LS194

Commit message: Alu control and modules completed, as well as Stack pointer module
Parts:
- D1, D2, D3, D4, D5, D6, D7, D8: value LED -> RED
Changed lines of the file:
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@@
 			)
 		)
-		(property "Value" "LED"
+		(property "Value" "RED"
 			(at 168.91 91.7574 90)
 			(effects
@@
 			)
 		)
-		(property "Value" "LED"
+		(property "Value" "RED"
 			(at 142.24 91.7574 90)
 			(effects
@@
 			)
 		)
-		(property "Value" "LED"
+		(property "Value" "RED"
 			(at 151.13 91.7574 90)
 			(effects
@@
 			)
 		)
-		(property "Value" "LED"
+		(property "Value" "RED"
 			(at 133.35 91.7574 90)
 			(effects
@@
 			)
 		)
-		(property "Value" "LED"
+		(property "Value" "RED"
 			(at 124.46 91.7574 90)
 			(effects
@@
 			)
 		)
-		(property "Value" "LED"
+		(property "Value" "RED"
 			(at 106.68 91.7574 90)
 			(effects
@@
 			)
 		)
-		(property "Value" "LED"
+		(property "Value" "RED"
 			(at 160.02 91.7574 90)
 			(effects
@@
 			)
 		)
-		(property "Value" "LED"
+		(property "Value" "RED"
 			(at 115.57 91.7574 90)
 			(effects

Commit message: Last revision of the cpu, all boards have been ordered. Implementation to be tested and documented in following commits.
Parts:
- renumbered R8 to R10, R1 to R3, R2 to R4, R3 to R5, R4 to R6, R5 to R7, R6 to R8, R7 to R9, U1 to U4, U2 to U5, U3 to U6
Connections:
- net MR renamed ~{MR}
Other:
- moved on the sheet: D1, D2, D3, D4, D5, D6, D7, D8, R10, R3, R4, R5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
