File: 04_Memory Modules/mar_register.kicad_sch (KiCad schematic)
At the start: 40 parts, among them U1 74LS139, U2 74LS08, U3 74LS193, U4 74LS245, U5 74LS193, U6 74LS193, U7 74LS245, U8 74LS193

Commit message: Last revision of the cpu, all boards have been ordered. Implementation to be tested and documented in following commits.
Parts:
- removed U1: 74LS139, Package_DIP:DIP-16_W7.62mm, symbol 74xx:74LS139
- removed U2: 74LS08, Package_DIP:DIP-14_W7.62mm, symbol 74xx:74LS08
- removed U3, U5, U6, U8: 74LS193, Package_DIP:DIP-16_W7.62mm, symbol 74xx:74LS193
- added C1, C2, C3, C4, C5, C6: 100n, Capacitor_THT:C_Disc_D4.7mm_W2.5mm_P5.00mm, symbol Device:C
- added U1, U3, U4, U6: 74LS161, Package_DIP:DIP-16_W7.62mm, symbol 74xx:74LS161
- added U9: 74LS04, Package_DIP:DIP-14_W7.62mm, symbol 74xx:74LS04
- renumbered U4 to U2, U7 to U5
Connections:
- net CLK: now also U1.2 (CP), U3.2 (CP), U4.2 (CP), U6.2 (CP)
- net D0: now also U1.3 (D0), U4.3 (D0)
- net D1: now also U1.4 (D1), U4.4 (D1)
- net D2: now also U1.5 (D2), U4.5 (D2)
- net D3: now also U1.6 (D3), U4.6 (D3)
- net D4: now also U3.3 (D0), U6.3 (D0)
- net D5: now also U3.4 (D1), U6.4 (D1)
- net D6: now also U3.5 (D2), U6.5 (D2)
- net D7: now also U3.6 (D3), U6.6 (D3)
- net GND: now also C1.2, C2.2, C3.2, C4.2, C5.2, C6.2, U1.8 (GND), U3.8 (GND), U4.8 (GND), U6.8 (GND)
- net VCC: now also C1.1, C2.1, C3.1, C4.1, C5.1, C6.1, U1.16 (VCC), U3.16 (VCC), U4.16 (VCC), U6.16 (VCC)
- net ~{MLI}: now also U1.9 (~{PE}), U3.9 (~{PE})
- net ~{MMI}: now also U4.9 (~{PE}), U6.9 (~{PE})
- net at D1.2 (A), U2.2 (A0): now also U1.14 (Q0)
- net at D14.2 (A), U5.7 (A5): now also U6.13 (Q1)
- net at D2.2 (A), U2.3 (A1): now also U1.13 (Q1)
- net at D3.2 (A), U2.4 (A2): now also U1.12 (Q2)
- net at D10.2 (A), U5.3 (A1): now also U4.13 (Q1)
- net at D9.2 (A), U5.2 (A0): now also U4.14 (Q0)
- net at D11.2 (A), U5.4 (A2): now also U4.12 (Q2)
- net at D12.2 (A), U5.5 (A3): now also U4.11 (Q3)
- net at D13.2 (A), U5.6 (A4): now also U6.14 (Q0)
- net at D15.2 (A), U5.8 (A6): now also U6.12 (Q2)
- net at D16.2 (A), U5.9 (A7): now also U6.11 (Q3)
- net at D6.2 (A), U2.7 (A5): now also U3.13 (Q1)
- net at D5.2 (A), U2.6 (A4): now also U3.14 (Q0)
- net at D7.2 (A), U2.8 (A6): now also U3.12 (Q2)
- net at D8.2 (A), U2.9 (A7): now also U3.11 (Q3)
- net at D4.2 (A), U2.5 (A3): now also U1.11 (Q3)
- new net: U1.1 (~{MR}), U3.1 (~{MR}), U4.1 (~{MR}), U6.1 (~{MR}), U9.4
- new net: U3.15 (TC), U4.7 (CEP)
- new net: U1.15 (TC), U3.7 (CEP)
- new net: U4.15 (TC), U6.7 (CEP)
- new net MAR: U9.3
- new net MCE: U1.10 (CET), U1.7 (CEP), U3.10 (CET), U4.10 (CET), U6.10 (CET)
- no-connect marks 7 -> 1
Other:
- note added: "Decoupling cap"
- note added: "Memory Address Register"
- note removed: "16-bit counter register"
- note removed: "Function selector (INC/DEC/CLR)"
- note removed: "Power supply"
- note removed: "Unused decoder"
- moved on the sheet: D1, D10, D11, D12, D13, D14, D15, D16, D2, D3, D4, D5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
