File: 04_Memory Modules/ram.kicad_sch (KiCad schematic)
At the start: 5 parts, among them Q1 PN2222A, U10 CY7C199, U9 CY7C199

Commit message: Last revision of the cpu, all boards have been ordered. Implementation to be tested and documented in following commits.
Parts:
- removed Q1: PN2222A, Package_TO_SOT_THT:TO-92_Inline, symbol Transistor_BJT:PN2222A
- removed R17: 1K, Resistor_THT:R_Axial_DIN0207_L6.3mm_D2.5mm_P10.16mm_Horizontal, symbol Device:R_US
- removed R18: 10K, Resistor_THT:R_Axial_DIN0207_L6.3mm_D2.5mm_P10.16mm_Horizontal, symbol Device:R_US
- added C7, C8, C9: 100n, Capacitor_THT:C_Disc_D4.7mm_W2.5mm_P5.00mm, symbol Device:C
- added U9: 74LS04, Package_DIP:DIP-14_W7.62mm, symbol 74xx:74LS04
- renumbered U9 to U7, U10 to U8
Connections:
- net A15: now also U9.1
- net GND: now also C7.2, C8.2, C9.2, U9.11, U9.13, U9.5, U9.7 (GND), U9.9
- net VCC: now also C7.1, C8.1, C9.1, U9.14 (VCC)
- net at U8.20 (~{CE}): now also U9.2
- no-connect marks 0 -> 4
Other:
- note added: "Decoupling cap"
- note added: "Power Supply"
- note added: "Unused Ports"
- moved on the sheet: U7, U8
