File: 04_Memory Modules/rom.kicad_sch (KiCad schematic)
At the start: 1 part, among them U11 28C256

Commit message: Last revision of the cpu, all boards have been ordered. Implementation to be tested and documented in following commits.
Parts:
- added C10: 10nF, Capacitor_THT:C_Disc_D4.7mm_W2.5mm_P5.00mm, symbol Device:C
- renumbered U11 to U10
Connections:
- net GND: now also C10.2
- net VCC: now also C10.1
Other:
- note added: "Decoupling cap"
Changed lines of the file:
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@@
+		)
+	)
+	(text "Decoupling cap"
+		(exclude_from_sim no)
+		(at 212.598 61.214 0)
+		(effects
+			(font
+				(size 2.54 2.54)
+			)
 		)
 	)
@@
 	(wire
 		(pts
+			(xy 208.28 68.58) (xy 208.28 72.39)
+		)
+		(stroke
+			(width 0)
+			(type default)
+		)
+	)
+	(wire
+		(pts
 			(xy 157.48 100.33) (xy 157.48 102.87)
 		)
@@
 	(wire
 		(pts
+			(xy 214.63 76.2) (xy 215.9 76.2)
+		)
+		(stroke
+			(width 0)
+			(type default)
+		)
+	)
+	(wire
+		(pts
 			(xy 121.92 77.47) (xy 121.92 80.01)
 		)
@@
 	(wire
 		(pts
+			(xy 209.55 68.58) (xy 208.28 68.58)
+		)
+		(stroke
+			(width 0)
+			(type default)
+		)
+	)
+	(wire
+		(pts
 			(xy 162.56 100.33) (xy 162.56 102.87)
 		)
@@
 		(pts
 			(xy 129.54 100.33) (xy 129.54 102.87)
+		)
+		(stroke
+			(width 0)
+			(type default)
+		)
+	)
+	(wire
+		(pts
+			(xy 215.9 72.39) (xy 215.9 76.2)
 		)
 		(stroke
@@
 		(shape tri_state)
 		(at 129.54 77.47 90)
+		(effects
+			(font
+				(size 1.27 1.27)
+			)
+			(justify left)
+		)
+	)
+	(hierarchical_label "GND"
+		(shape input)
+		(at 214.63 76.2 180)
+		(effects
+			(font
+				(size 1.27 1.27)
+			)
+			(justify right)
+		)
+	)
+	(hierarchical_label "VCC"
+		(shape input)
+		(at 209.55 68.58 0)
 		(effects
 			(font
@@
 		(on_board yes)
 		(dnp no)
-		(fields_autoplaced yes)
-		(property "Reference" "U11"
-			(at 109.22 84.7246 90)
+		(property "Reference" "U10"
+			(at 139.446 88.646 90)
 			(effects
 				(font
@@
 		)
 		(property "Value" "28C256"
-			(at 109.22 87.2646 90)
+			(at 139.446 91.186 90)
 			(effects
 				(font
@@
 			(project "03_Memory"
 				(path "/67f85d1f-fa07-4d32-87fd-2c14cd08dcf9/5d6cf42f-491f-45f7-834b-b917429b208c"
-					(reference "U11")
+					(reference "U10")
 					(unit 1)
 				)
+			)
+		)
+	)
+	(symbol
+		(lib_id "Device:C")
+		(at 212.09 72.39 90)
+		(unit 1)
+		(exclude_from_sim no)
+		(in_bom yes)
+		(on_board yes)
+		(dnp no)
+		(property "Reference" "C10"
+			(at 218.694 70.866 90)
+			(effects
+				(font
+					(size 1.27 1.27)
+				)
+				(justify right)
+			)
+		)
+		(property "Value" "10nF"
+			(at 218.694 73.406 90)
+			(effects
+				(font
+					(size 1.27 1.27)
+				)
+				(justify right)
+			)
+		)
+		(property "Footprint" "Capacitor_THT:C_Disc_D4.7mm_W2.5mm_P5.00mm"
+			(at 215.9 71.4248 0)
+			(effects
+				(font
+					(size 1.27 1.27)
+				)
+				(hide yes)
+			)
+		)
+		(property "Datasheet" "~"
+			(at 212.09 72.39 0)
+			(effects
+				(font
+					(size 1.27 1.27)
+				)
+				(hide yes)
+			)
+		)
+		(property "Description" "Unpolarized capacitor"
+			(at 212.09 72.39 0)
+			(effects
+				(font
+					(size 1.27 1.27)
+				)
+				(hide yes)
+			)
+		)
+		(pin "2"
+		)
+		(pin "1"
+		)
+		(instances
+			(project "Memory Modules"
+				(path "/67f85d1f-fa07-4d32-87fd-2c14cd08dcf9/5d6cf42f-491f-45f7-834b-b917429b208c"
+					(reference "C10")
+					(unit 1)
+				)
