File: 05_Program Counter/Program Counter.kicad_pcb (KiCad board)
At the start: 2 copper layers, 100 x 100 mm, 55 parts, among them J1 Data Out 1, J2 Data Out 2, J3 Address Out 1, J4 Address Out 2, J5 Data bus, J6 Address Bus 1, J7 Address Bus 2, J8 Input 1, J9 Input 2, U1 74LS161, U10 74LS138, U2 74LS245, U3 74LS161, U4 74LS161, U5 74LS245, U6 74LS161, U7 74LS138, U8 74LS138, U9 74LS138

Commit message: Last revision of the cpu, all boards have been ordered. Implementation to be tested and documented in following commits.
Parts:
- removed the J2 at (116.0, 77.1)
- removed the J3 at (104.2, 54.2)
- removed the J4 at (104.2, 77.1)
- added C1: 100n, Capacitor_THT:C_Disc_D3.0mm_W1.6mm_P2.50mm, F.Cu at (34.6, 103.1)
- added C10: 100n, Capacitor_THT:C_Disc_D3.0mm_W1.6mm_P2.50mm, F.Cu at (84.2, 56.8)
- added C11: 100n, Capacitor_THT:C_Disc_D3.0mm_W1.6mm_P2.50mm, F.Cu at (84.1, 79.5)
- added C2: 100n, Capacitor_THT:C_Disc_D3.0mm_W1.6mm_P2.50mm, F.Cu at (97.7, 41.6)
- added C3: 100n, Capacitor_THT:C_Disc_D3.0mm_W1.6mm_P2.50mm, F.Cu at (32.5, 54.4)
- added C4: 100n, Capacitor_THT:C_Disc_D3.0mm_W1.6mm_P2.50mm, F.Cu at (34.4, 74.1)
- added C5: 100n, Capacitor_THT:C_Disc_D3.0mm_W1.6mm_P2.50mm, F.Cu at (51.1, 104.2)
- added C6: 100n, Capacitor_THT:C_Disc_D3.0mm_W1.6mm_P2.50mm, F.Cu at (62.7, 56.4)
- added C7: 100n, Capacitor_THT:C_Disc_D3.0mm_W1.6mm_P2.50mm, F.Cu at (57.0, 79.1)
- added C8: 100n, Capacitor_THT:C_Disc_D3.0mm_W1.6mm_P2.50mm, F.Cu at (95.9, 54.3)
- added C9: 100n, Capacitor_THT:C_Disc_D3.0mm_W1.6mm_P2.50mm, F.Cu at (95.8, 79.1)
- added U2: 74LS04, Package_DIP:DIP-14_W7.62mm, F.Cu at (100.3, 49.2)
- J1: value Data Out 1 -> Data-Address Out; footprint Custom:PinHeader_1x08_P2.54mm_Vertical -> Connector_PinHeader_2.54mm:PinHeader_2x16_P2.54mm_Horizontal
- moved J1 7.62 mm to (108.6, 54.1)
- renumbered J5 to J2, J6 to J3, J7 to J4, J8 to J5, J9 to J6, U9 to U10, U10 to U11, U2 to U3, U3 to U4, U4 to U5, U5 to U6, U6 to U7, U7 to U8, U8 to U9
Connections:
- net /A0 renamed A0
- net /A1 renamed A1
- net /A10 renamed A10
- net /A11 renamed A11
- net /A12 renamed A12
- net /A13 renamed A13
- net /A14 renamed A14
- net /A15 renamed A15
- net /A2 renamed A2
- net /A3 renamed A3
- net /A4 renamed A4
- net /A5 renamed A5
- net /A6 renamed A6
- net /A7 renamed A7
- net /A8 renamed A8
- net /A9 renamed A9
- net /AC0 renamed AC0
- net /AC1 renamed AC1
- net /AC2 renamed AC2
- net /AC3 renamed AC3
- net /D0 renamed D0
- net /D1 renamed D1
- net /D2 renamed D2
- net /D3 renamed D3
- net /D4 renamed D4
- net /D5 renamed D5
- net /D6 renamed D6
- net /D7 renamed D7
- net /DC0 renamed DC0
- net /DC1 renamed DC1
- net /DC2 renamed DC2
- net /DC3 renamed DC3
- net /PCE renamed PCE
- net /VCC renamed VCC
- net /~{PCO} renamed ~{PCO}
- net /~{PLI} renamed ~{PLI}
- net /~{PMI} renamed ~{PMI}
- J1 pad 2: /Data-Bus Out Selector/O1 -> /Addr-Bus Out Selector/O0
- J1 pad 3: /Data-Bus Out Selector/O2 -> /Data-Bus Out Selector/O1
- J1 pad 4: /Data-Bus Out Selector/O3 -> /Addr-Bus Out Selector/O1
- J1 pad 5: /Data-Bus Out Selector/O4 -> /Data-Bus Out Selector/O2
- J1 pad 6: /Data-Bus Out Selector/O5 -> /Addr-Bus Out Selector/O2
- J1 pad 7: /Data-Bus Out Selector/O6 -> /Data-Bus Out Selector/O3
- J1 pad 8: /Data-Bus Out Selector/O7 -> /Addr-Bus Out Selector/O3
- J5 pad 2: /CLK -> CLK
- J5 pad 7: /~{CLR} -> PCR
- J5 pad 8: /GND -> GND
- R1 pad 2: /GND -> GND
- R10 pad 2: /GND -> GND
- R11 pad 2: /GND -> GND
- R12 pad 2: /GND -> GND
- R13 pad 2: /GND -> GND
- R14 pad 2: /GND -> GND
- R15 pad 2: /GND -> GND
- R16 pad 2: /GND -> GND
- R2 pad 2: /GND -> GND
- R3 pad 2: /GND -> GND
- R4 pad 2: /GND -> GND
- R5 pad 2: /GND -> GND
- R6 pad 2: /GND -> GND
- R7 pad 2: /GND -> GND
- R8 pad 2: /GND -> GND
- R9 pad 2: /GND -> GND
- U1 pad 1: /~{CLR} -> Net-(U1-~{MR})
- U1 pad 2: /CLK -> CLK
- U1 pad 8: /GND -> GND
- U10 pad 8: /CLK -> GND
- U11 pad 4: /CLK -> GND
- U11 pad 5: /CLK -> GND
- U11 pad 8: /CLK -> GND
- U3 pad 10: /GND -> GND
- U4 pad 1: /~{CLR} -> Net-(U1-~{MR})
- U4 pad 2: /CLK -> CLK
- U4 pad 8: /GND -> GND
- U5 pad 1: /~{CLR} -> Net-(U1-~{MR})
- U5 pad 2: /CLK -> CLK
- U5 pad 8: /GND -> GND
- U6 pad 10: /GND -> GND
- U7 pad 1: /~{CLR} -> Net-(U1-~{MR})
- U7 pad 2: /CLK -> CLK
- U7 pad 8: /GND -> GND
- U8 pad 8: /CLK -> GND
- U9 pad 4: /CLK -> GND
- U9 pad 5: /CLK -> GND
- U9 pad 8: /CLK -> GND
Routing:
- net /CLK: track 180.3 -> 0.00 mm, vias 5 -> 0
- net GND: track 0.00 -> 155.9 mm, vias 0 -> 4
- net Net-(U1-~{MR}): track 0.00 -> 127.4 mm, vias 0 -> 5
- net /~{CLR}: track 127.3 -> 0.00 mm, vias 5 -> 0
- net CLK: track 0.00 -> 120.5 mm, vias 0 -> 4
- net /GND: track 100.8 -> 0.00 mm, vias 2 -> 0
- net VCC: track 279.0 -> 310.5 mm
- net PCR: track 0.00 -> 27.0 mm, vias 0 -> 2
- net /Addr-Bus Out Selector/O15: track 44.9 -> 53.9 mm, vias 3 -> 4
- net /Addr-Bus Out Selector/O10: track 30.8 -> 39.8 mm
- net /Addr-Bus Out Selector/O8: track 31.1 -> 40.1 mm
- net /Addr-Bus Out Selector/O9: track 30.6 -> 39.6 mm
- net /Addr-Bus Out Selector/O11: track 31.0 -> 39.9 mm
- net /Addr-Bus Out Selector/O13: track 31.1 -> 40.0 mm
- net /Addr-Bus Out Selector/O14: track 31.2 -> 40.1 mm
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- added copper zone on B.Cu, net GND
- removed copper zone on B.Cu, net /GND
Other:
- board text added: "Program Counter and Bus Out Selector v1.2"
- board text removed: "Program Counter and Bus Out Selector v1.1"
