File: 05_Program Counter/data-selector.kicad_sch (KiCad schematic)
At the start: 2 parts, among them U7 74LS138, U8 74LS138

Commit message: Last revision of the cpu, all boards have been ordered. Implementation to be tested and documented in following commits.
Parts:
- added C8, C9: 100n, Capacitor_THT:C_Disc_D3.0mm_W1.6mm_P2.50mm, symbol Device:C
- renumbered U7 to U8, U8 to U9
Connections:
- net GND: now also C8.2, C9.2
- net VCC: now also C8.1, C9.1
Other:
- note added: "Decoupling cap"
Changed lines of the file:
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@@
 	(generator_version "9.0")
 	(paper "A4")
+	(text "Decoupling cap"
+		(exclude_from_sim no)
+		(at 240.538 47.244 0)
+		(effects
+			(font
+				(size 2.54 2.54)
+			)
+		)
+	)
 	(text "LSB bus selector"
 		(exclude_from_sim no)
@@
 			)
 		)
+	)
+	(junction
+		(at 243.84 67.31)
+		(diameter 0)
+		(color 0 0 0 0)
 	)
 	(junction
@@
 	)
 	(junction
+		(at 236.22 59.69)
+		(diameter 0)
+		(color 0 0 0 0)
+	)
+	(junction
 		(at 160.02 82.55)
 		(diameter 0)
@@
 	(wire
 		(pts
+			(xy 236.22 55.88) (xy 236.22 59.69)
+		)
+		(stroke
+			(width 0)
+			(type default)
+		)
+	)
+	(wire
+		(pts
 			(xy 114.3 77.47) (xy 116.84 77.47)
 		)
@@
 	(wire
 		(pts
+			(xy 242.57 71.12) (xy 243.84 71.12)
+		)
+		(stroke
+			(width 0)
+			(type default)
+		)
+	)
+	(wire
+		(pts
 			(xy 114.3 80.01) (xy 116.84 80.01)
 		)
@@
 	(wire
 		(pts
+			(xy 243.84 59.69) (xy 243.84 67.31)
+		)
+		(stroke
+			(width 0)
+			(type default)
+		)
+	)
+	(wire
+		(pts
 			(xy 160.02 82.55) (xy 160.02 85.09)
 		)
@@
 	(wire
 		(pts
+			(xy 237.49 55.88) (xy 236.22 55.88)
+		)
+		(stroke
+			(width 0)
+			(type default)
+		)
+	)
+	(wire
+		(pts
 			(xy 157.48 69.85) (xy 160.02 69.85)
 		)
@@
 	(wire
 		(pts
+			(xy 243.84 67.31) (xy 243.84 71.12)
+		)
+		(stroke
+			(width 0)
+			(type default)
+		)
+	)
+	(wire
+		(pts
 			(xy 86.36 72.39) (xy 88.9 72.39)
 		)
@@
 		)
 	)
+	(wire
+		(pts
+			(xy 236.22 59.69) (xy 236.22 67.31)
+		)
+		(stroke
+			(width 0)
+			(type default)
+		)
+	)
 	(hierarchical_label "C3"
 		(shape input)
@@
 		)
 	)
+	(hierarchical_label "GND"
+		(shape input)
+		(at 242.57 71.12 180)
+		(effects
+			(font
+				(size 1.27 1.27)
+			)
+			(justify right)
+		)
+	)
 	(hierarchical_label "O8"
 		(shape output)
@@
 		)
 	)
+	(hierarchical_label "VCC"
+		(shape input)
+		(at 237.49 55.88 0)
+		(effects
+			(font
+				(size 1.27 1.27)
+			)
+			(justify left)
+		)
+	)
 	(hierarchical_label "O14"
 		(shape output)
@@
 			)
 			(justify right)
+		)
+	)
+	(symbol
+		(lib_id "Device:C")
+		(at 240.03 67.31 90)
+		(unit 1)
+		(exclude_from_sim no)
+		(in_bom yes)
+		(on_board yes)
+		(dnp no)
+		(property "Reference" "C9"
+			(at 246.634 65.786 90)
+			(effects
+				(font
+					(size 1.27 1.27)
+				)
+				(justify right)
+			)
+		)
+		(property "Value" "100n"
+			(at 246.634 68.326 90)
+			(effects
+				(font
+					(size 1.27 1.27)
+				)
+				(justify right)
+			)
+		)
+		(property "Footprint" "Capacitor_THT:C_Disc_D3.0mm_W1.6mm_P2.50mm"
+			(at 243.84 66.3448 0)
+			(effects
+				(font
+					(size 1.27 1.27)
+				)
+				(hide yes)
+			)
+		)
+		(property "Datasheet" "~"
+			(at 240.03 67.31 0)
+			(effects
+				(font
+					(size 1.27 1.27)
+				)
+				(hide yes)
+			)
+		)
+		(property "Description" "Unpolarized capacitor"
+			(at 240.03 67.31 0)
+			(effects
+				(font
+					(size 1.27 1.27)
+				)
+				(hide yes)
+			)
+		)
+		(pin "2"
+		)
+		(pin "1"
+		)
+		(instances
+			(project "Program Counter"
+				(path "/276e8094-1ce6-4ca8-b69c-ac07ef6e83aa/08bb57c0-efe9-4381-8465-59433d2dda0c"
+					(reference "C9")
+					(unit 1)
+				)
+				(path "/276e8094-1ce6-4ca8-b69c-ac07ef6e83aa/f9a8d2b2-a7a4-4257-8637-a0121ba4aaef"
+					(reference "C11")
+					(unit 1)
+				)
+			)
 		)
 	)
@@
 		(dnp no)
 		(fields_autoplaced yes)
-		(property "Reference" "U8"
+		(property "Reference" "U9"
 			(at 174.8633 59.69 0)
 			(effects
@@
 			(project "04_Program Counter"
 				(path "/276e8094-1ce6-4ca8-b69c-ac07ef6e83aa/08bb57c0-efe9-4381-8465-59433d2dda0c"
-					(reference "U8")
+					(reference "U9")
 					(unit 1)
 				)
 				(path "/276e8094-1ce6-4ca8-b69c-ac07ef6e83aa/f9a8d2b2-a7a4-4257-8637-a0121ba4aaef"
-					(reference "U10")
+					(reference "U11")
+					(unit 1)
+				)
+			)
+		)
+	)
+	(symbol
+		(lib_id "Device:C")
+		(at 240.03 59.69 90)
+		(unit 1)
+		(exclude_from_sim no)
+		(in_bom yes)
+		(on_board yes)
+		(dnp no)
+		(property "Reference" "C8"
+			(at 246.634 58.166 90)
+			(effects
+				(font
+					(size 1.27 1.27)
+				)
+				(justify right)
+			)
+		)
+		(property "Value" "100n"
+			(at 246.634 60.706 90)
+			(effects
+				(font
+					(size 1.27 1.27)
+				)
+				(justify right)
+			)
+		)
+		(property "Footprint" "Capacitor_THT:C_Disc_D3.0mm_W1.6mm_P2.50mm"
+			(at 243.84 58.7248 0)
+			(effects
+				(font
+					(size 1.27 1.27)
+				)
+				(hide yes)
+			)
+		)
+		(property "Datasheet" "~"
+			(at 240.03 59.69 0)
+			(effects
+				(font
+					(size 1.27 1.27)
+				)
+				(hide yes)
+			)
+		)
+		(property "Description" "Unpolarized capacitor"
+			(at 240.03 59.69 0)
+			(effects
+				(font
+					(size 1.27 1.27)
+				)
+				(hide yes)
+			)
+		)
+		(pin "2"
+		)
+		(pin "1"
+		)
+		(instances
+			(project "Program Counter"
+				(path "/276e8094-1ce6-4ca8-b69c-ac07ef6e83aa/08bb57c0-efe9-4381-8465-59433d2dda0c"
+					(reference "C8")
+					(unit 1)
+				)
+				(path "/276e8094-1ce6-4ca8-b69c-ac07ef6e83aa/f9a8d2b2-a7a4-4257-8637-a0121ba4aaef"
+					(reference "C10")
 					(unit 1)
 				)
@@
 		(dnp no)
 		(fields_autoplaced yes)
-		(property "Reference" "U7"
+		(property "Reference" "U8"
 			(at 103.7433 59.69 0)
 			(effects
@@
 			(project "04_Program Counter"
 				(path "/276e8094-1ce6-4ca8-b69c-ac07ef6e83aa/08bb57c0-efe9-4381-8465-59433d2dda0c"
-					(reference "U7")
+					(reference "U8")
 					(unit 1)
 				)
 				(path "/276e8094-1ce6-4ca8-b69c-ac07ef6e83aa/f9a8d2b2-a7a4-4257-8637-a0121ba4aaef"
-					(reference "U9")
+					(reference "U10")
 					(unit 1)
 				)
