File: 06_Instruction Register/sequencer.kicad_sch (KiCad schematic)
At the start: 9 parts, among them U3 74LS161

Commit message: Last revision of the cpu, all boards have been ordered. Implementation to be tested and documented in following commits.
Parts:
- added C3, C4: 100n, Capacitor_THT:C_Disc_D3.0mm_W1.6mm_P2.50mm, symbol Device:C
- added U4: 74LS04, Package_DIP:DIP-14_W7.62mm, symbol 74xx:74LS04
Connections:
- net GND: now also C3.2, C4.2, U4.11, U4.13, U4.3, U4.5, U4.7 (GND), U4.9
- net VCC: now also C3.1, C4.1, U4.14 (VCC)
- net ~{SSR}: no longer names the net of U3.1 (~{MR})
- net ~{SSR}: now also U4.2
- new net SSR: U4.1
- no-connect marks 5 -> 10
Other:
- note added: "Decoupling cap"
